File: pcb/miku/miku.kicad_sch (KiCad schematic)
At the start: 17 parts, among them J01 MIDI_IN, J02 PITCH_CV_IN, J03 GATE_IN, J04 VOL_CV_IN, J05 SYLL_CV_IN, J06 PORT_CV_IN, J07 TBD_IN, J08 VIBTYPE_CV_IN, J09 VIBRATE_CV_IN, J10 VIBDELAY_CV_IN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

Commit message: initial cut, v0.1.0-alpha
Parts:
- IX02: renamed from IX03; value BOTTOM_INTERCONNECT -> TOP_INTERCONNECT
- IX03: renamed from IX02; value TOP_INTERCONNECT -> BOTTOM_INTERCONNECT
Connections:
- net VIBRATE_CV_IN: now also IX03.6 (Pin_6); no longer IX03.8 (Pin_8)
- net VOL_CV_IN: now also IX03.8 (Pin_8); no longer IX03.6 (Pin_6)
Changed lines of the file:
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@@
 	(wire
 		(pts
-			(xy 45.72 34.29) (xy 88.9 34.29)
+			(xy 45.72 40.64) (xy 120.65 40.64)
 		)
 		(stroke
@@
 	(wire
 		(pts
+			(xy 76.2 34.29) (xy 88.9 34.29)
+		)
+		(stroke
+			(width 0)
+			(type default)
+		)
+	)
+	(wire
+		(pts
 			(xy 138.43 46.99) (xy 138.43 29.21)
 		)
@@
 	(wire
 		(pts
+			(xy 101.6 24.13) (xy 120.65 24.13)
+		)
+		(stroke
+			(width 0)
+			(type default)
+		)
+	)
+	(wire
+		(pts
 			(xy 101.6 26.67) (xy 118.11 26.67)
 		)
@@
 	(wire
 		(pts
+			(xy 76.2 45.72) (xy 76.2 34.29)
+		)
+		(stroke
+			(width 0)
+			(type default)
+		)
+	)
+	(wire
+		(pts
 			(xy 135.89 44.45) (xy 135.89 26.67)
 		)
@@
 	(wire
 		(pts
-			(xy 101.6 24.13) (xy 120.65 24.13)
+			(xy 76.2 45.72) (xy 120.65 45.72)
 		)
 		(stroke
@@
 	(wire
 		(pts
+			(xy 120.65 40.64) (xy 120.65 24.13)
+		)
+		(stroke
+			(width 0)
+			(type default)
+		)
+	)
+	(wire
+		(pts
 			(xy 16.51 173.99) (xy 30.48 173.99)
 		)
@@
 	(wire
 		(pts
-			(xy 120.65 152.4) (xy 120.65 24.13)
-		)
-		(stroke
-			(width 0)
-			(type default)
-		)
-	)
-	(wire
-		(pts
-			(xy 45.72 77.47) (xy 45.72 34.29)
+			(xy 120.65 152.4) (xy 120.65 45.72)
+		)
+		(stroke
+			(width 0)
+			(type default)
+		)
+	)
+	(wire
+		(pts
+			(xy 45.72 77.47) (xy 45.72 40.64)
 		)
 		(stroke
@@
 	)
 	(label "VIBRATE_CV_IN"
-		(at 101.6 24.13 0)
+		(at 76.2 34.29 0)
 		(fields_autoplaced yes)
 		(effects
@@
 		)
 	)
+	(label "VOL_CV_IN"
+		(at 101.6 24.13 0)
+		(fields_autoplaced yes)
+		(effects
+			(font
+				(size 1.27 1.27)
+			)
+			(justify left bottom)
+		)
+	)
 	(label "SYLL_CV_IN"
 		(at 101.6 34.29 0)
@@
 	(label "GATE_IN"
 		(at 80.01 31.75 0)
-		(fields_autoplaced yes)
-		(effects
-			(font
-				(size 1.27 1.27)
-			)
-			(justify left bottom)
-		)
-	)
-	(label "VOL_CV_IN"
-		(at 78.74 34.29 0)
 		(fields_autoplaced yes)
 		(effects
@@
 		(dnp no)
 		(fields_autoplaced yes)
-		(property "Reference" "IX02"
+		(property "Reference" "IX03"
 			(at 95.25 15.24 0)
 			(effects
@@
 			)
 		)
-		(property "Value" "TOP_INTERCONNECT"
+		(property "Value" "BOTTOM_INTERCONNECT"
 			(at 95.25 17.78 0)
 			(effects
@@
 			(project "miku"
 				(path "/ebb7bf49-4f3a-4d48-a7af-62f1e8931a47"
-					(reference "IX02")
+					(reference "IX03")
 					(unit 1)
 				)
@@
 		(dnp no)
 		(fields_autoplaced yes)
-		(property "Reference" "IX03"
+		(property "Reference" "IX02"
 			(at 144.78 64.77 0)
 			(effects
@@
 			)
 		)
-		(property "Value" "BOTTOM_INTERCONNECT"
+		(property "Value" "TOP_INTERCONNECT"
 			(at 144.78 67.31 0)
 			(effects
@@
 			(project "miku"
 				(path "/ebb7bf49-4f3a-4d48-a7af-62f1e8931a47"
-					(reference "IX03")
+					(reference "IX02")
 					(unit 1)
 				)
