File: pcb/miku/miku.kicad_pcb (KiCad board)
At the start: 2 copper layers, 71.1 x 108 mm, 24 parts, among them J01 MIDI_IN, J02 PITCH_CV_IN, J03 GATE_IN, J04 VOL_CV_IN, J05 SYLL_CV_IN, J06 PORT_CV_IN, J07 TBD_IN, J08 VIBTYPE_CV_IN, J09 VIBRATE_CV_IN, J10 VIBDELAY_CV_IN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

Commit message: initial cut, v0.1.0-alpha
Parts:
- added G***: LOGO, portal-marks:portal-logo-eye-door-95mm, B.Cu at (110.5, 116.5)
- IX01: value SCREEN_INTERCONNECT -> MEDIA_INTERCONNECT; footprint Connector_PinHeader_2.54mm:PinHeader_1x04_P2.54mm_Vertical -> Connector_PinHeader_2.54mm:PinHeader_2x04_P2.54mm_Vertical; moved to F.Cu
- moved IX01 8.18 mm to (106.4, 62.5)
- moved J11 1.22 mm to (105.0, 92.0)
- moved J12 1.22 mm to (116.0, 92.0)
- moved IX03 0.50 mm to (117.6, 143.5)
Routing:
- net (no net): track 0.00 -> 1876.0 mm
Other:
- board text added: "${COMPANY}"
- board text added: "${REVISION}"
- board text added: "${TITLE}"

Commit message: Silkscreened the IX pinouts
Parts:
- IX01: renamed from IX02; value TOP_INTERCONNECT -> TOP_IX
- IX02: renamed from IX01; value MEDIA_INTERCONNECT -> MEDIA_IX; moved to B.Cu
- IX03: value BOTTOM_INTERCONNECT -> BOTTOM_IX
- moved IX02 7.66 mm to (114.1, 62.5)
Other:
- board text added: "3.3VA"
- board text added: "AUDL"
- board text added: "AUDR"
- board text added: "PITCH"
- board text added: "PORTM"
- board text added: "SCRN"
- board text added: "SYLL"
- board text added: "VIBDL"
- board text added: "VIBRT"
- board text added: "VIBTP"
- board text added: "VOLUM"
- board text added: "望"

Commit message: Revert "Added silkscreen labels for interconnect pins (#30)"
This reverts commit c19aa1e4f3f042fac9955cee06975aab86f3ba47.
Parts:
- IX01: renamed from IX02; value MEDIA_IX -> MEDIA_INTERCONNECT; moved to F.Cu
- IX02: renamed from IX01; value TOP_IX -> TOP_INTERCONNECT
- IX03: value BOTTOM_IX -> BOTTOM_INTERCONNECT
- moved IX01 7.66 mm to (106.4, 62.5)
Other:
- board text removed: "3.3VA"
- board text removed: "AUDL"
- board text removed: "AUDR"
- board text removed: "PITCH"
- board text removed: "PORTM"
- board text removed: "SCRN"
- board text removed: "SYLL"
- board text removed: "VIBDL"
- board text removed: "VIBRT"
- board text removed: "VIBTP"
- board text removed: "VOLUM"
- board text removed: "望"
